Commit message: Bug fixes

File: description/urdf/pioneer3dx.urdf (robot description, URDF)
Before this commit: robot pioneer3dx, 18 links, 17 joints
Links:
- link lms100: geometry collision box size=0.01 0.01 0.01; visual mesh filename=package://pioneer3dx_description/meshes/lms100.dae

File: description/urdf/pioneer3dx.xacro (robot description, xacro)
@@ -247,5 +247,5 @@
 			<origin xyz="0 0 0" rpy="0 0 0" />
 			<geometry>
-				<mesh filename="package://p3dx_description/meshes/lms100.dae" />
+				<mesh filename="package://pioneer3dx_description/meshes/lms100.dae" />
 			</geometry>
 		</visual>
